Commit message: feat : config and launchfile added for gripper replacement

File: xarm_description/urdf/xarm6_with_gripper.xacro (robot description, xacro)
@@ -13,6 +13,6 @@
     <xacro:arg name="rpy" default="0 0 0"/>
     <xacro:arg name="gripper_meshes_path" default=""/>
-    <xacro:arg name="rpy" default="0 0 0"/>
-    <xacro:arg name="xyz" default="0 0 0"/>
+    <xacro:arg name="tcp_z" default=""/>
+    <xacro:arg name="gripper_rpy" default="0 0 0"/>
     <!---->
     <!-- load xarm6 robot -->
@@ -24,12 +24,13 @@
                        effort_control="$(arg effort_control)" velocity_control="$(arg velocity_control)"
                        rs_d435i="$(arg add_realsense_d435i)" xyz="$(arg xyz)" rpy="$(arg rpy)"/>
+    <!-- load gripper -->
     <xacro:if value="$(arg add_realsense_d435i)">
         <xacro:load_gripper attach_to="$(arg prefix)link_eef" xyz="0 0 0.003" effort_control="$(arg effort_control)"
-                            velocity_control="$(arg velocity_control)" robot_dof="6"/>
+                            velocity_control="$(arg velocity_control)" robot_dof="6" />
     </xacro:if>
     <xacro:unless value="$(arg add_realsense_d435i)">
         <xacro:load_gripper attach_to="$(arg prefix)link_eef" effort_control="$(arg effort_control)"
-                            velocity_control="$(arg velocity_control)" robot_dof="6"
-                            gripper_meshes_path="$(arg gripper_meshes_path)"/>
+                            velocity_control="$(arg velocity_control)" robot_dof="6" rpy="$(arg gripper_rpy)"
+                            gripper_meshes_path="$(arg gripper_meshes_path)" tcp_z="$(arg tcp_z)"/>
     </xacro:unless>
     <xacro:if value="$(arg use_gazebo_camera)">

File: xarm_gripper/urdf/xarm_gripper.urdf.xacro (robot description, xacro)
@@ -5,7 +5,10 @@
     -->
     <xacro:macro name="xarm_gripper_urdf"
-                 params="prefix:='' attach_to:='' rpy:='0 0 0' xyz:='0 0 0' gripper_meshes_path:='' ">
+                 params="prefix:='' attach_to:='' rpy:='0 0 0' xyz:='0 0 0' gripper_meshes_path:='' tcp_z:='' ">
         <xacro:if value="${gripper_meshes_path == ''}">
             <xacro:property name="gripper_meshes_path" value="xarm_gripper/meshes"/>
+        </xacro:if>
+        <xacro:if value="${tcp_z == ''}">
+            <xacro:property name="tcp_z" value="0.172"/>
         </xacro:if>
         <xacro:unless value="${attach_to == ''}">
@@ -405,5 +408,5 @@
             type="fixed">
             <origin
-                xyz="0 0 0.172"
+                xyz="0 0 ${tcp_z}"
                 rpy="0 0 0"/>
             <parent

File: xarm_gripper/urdf/xarm_gripper_model.xacro (robot description, xacro)
@@ -10,9 +10,9 @@
     <xacro:macro name="load_gripper"
                  params="prefix:='' attach_to:='' ns:='xarm' xyz:='0 0 0' rpy:='0 0 0' effort_control:='false'
-                 velocity_control:='false' robot_dof:=7 gripper_meshes_path:='' ">
+                 velocity_control:='false' robot_dof:=7 gripper_meshes_path:='' tcp_z:='' ">
         <!-- gazebo plugin -->
         <!-- <xacro:gazebo_ros_control_plugin namespace="${ns}"/> -->
         <xacro:xarm_gripper_urdf prefix="${prefix}" attach_to="${attach_to}" xyz="${xyz}" rpy="${rpy}"
-                                 gripper_meshes_path="${gripper_meshes_path}"/>
+                                 gripper_meshes_path="${gripper_meshes_path}" tcp_z="${tcp_z}" />
         <xacro:xarm_gripper_transmission prefix="${prefix}"
                                          hard_interface="$(eval 'EffortJointInterface' if ${effort_control} else 'VelocityJointInterface' if ${velocity_control} else 'PositionJointInterface')"/>

Commit message: feat : upside_down and long_finger args added

File: xarm_description/urdf/xarm6_with_gripper.xacro (robot description, xacro)
@@ -10,9 +10,8 @@
     <xacro:arg name="use_gazebo_camera" default="false"/>
     <!--    added by me -->
-    <xacro:arg name="xyz" default="0 0 0"/>
-    <xacro:arg name="rpy" default="0 0 0"/>
     <xacro:arg name="gripper_meshes_path" default=""/>
-    <xacro:arg name="tcp_z" default=""/>
-    <xacro:arg name="gripper_rpy" default="0 0 0"/>
+    <xacro:arg name="base_link_rpy" default="0 0 0"/>
+    <xacro:arg name="base_link_xyz" default="0 0 0"/>
+    <xacro:arg name="long_finger" default="false"/>
     <!---->
     <!-- load xarm6 robot -->
@@ -20,17 +19,15 @@
     <!-- Attach gripper -->
     <xacro:include filename="$(find xarm_gripper)/urdf/xarm_gripper_model.xacro"/>
-    <!--    rpy and xyz added-->
     <xacro:xarm6_robot prefix="$(arg prefix)" namespace="$(arg ros_namespace)" limited="$(arg limited)"
                        effort_control="$(arg effort_control)" velocity_control="$(arg velocity_control)"
-                       rs_d435i="$(arg add_realsense_d435i)" xyz="$(arg xyz)" rpy="$(arg rpy)"/>
-    <!-- load gripper -->
+                       rs_d435i="$(arg add_realsense_d435i)" rpy="$(arg base_link_rpy)" xyz="$(arg base_link_xyz)"/>
     <xacro:if value="$(arg add_realsense_d435i)">
         <xacro:load_gripper attach_to="$(arg prefix)link_eef" xyz="0 0 0.003" effort_control="$(arg effort_control)"
-                            velocity_control="$(arg velocity_control)" robot_dof="6" />
+                            velocity_control="$(arg velocity_control)" robot_dof="6"/>
     </xacro:if>
     <xacro:unless value="$(arg add_realsense_d435i)">
         <xacro:load_gripper attach_to="$(arg prefix)link_eef" effort_control="$(arg effort_control)"
-                            velocity_control="$(arg velocity_control)" robot_dof="6" rpy="$(arg gripper_rpy)"
-                            gripper_meshes_path="$(arg gripper_meshes_path)" tcp_z="$(arg tcp_z)"/>
+                            velocity_control="$(arg velocity_control)" robot_dof="6"
+                            gripper_meshes_path="$(arg gripper_meshes_path)" long_finger="$(arg long_finger)"/>
     </xacro:unless>
     <xacro:if value="$(arg use_gazebo_camera)">

File: xarm_gripper/urdf/xarm_gripper.urdf.xacro (robot description, xacro)
@@ -5,16 +5,27 @@
     -->
     <xacro:macro name="xarm_gripper_urdf"
-                 params="prefix:='' attach_to:='' rpy:='0 0 0' xyz:='0 0 0' gripper_meshes_path:='' tcp_z:='' ">
+                 params="prefix:='' attach_to:='' gripper_meshes_path:='' long_finger:='false' upside_down:='false'">
+        <xacro:if value="${long_finger}">
+            <xacro:property name="gripper_meshes_path" value="xarm_gripper/meshes/xarm_long_finger_assembled"/>
+            <xacro:property name="tcp_offset_z" value="0.340"/>
+        </xacro:if>
+        <xacro:unless value="${long_finger}">
+            <xacro:property name="tcp_offset_z" value="0.172"/>
+        </xacro:unless>
         <xacro:if value="${gripper_meshes_path == ''}">
             <xacro:property name="gripper_meshes_path" value="xarm_gripper/meshes"/>
         </xacro:if>
-        <xacro:if value="${tcp_z == ''}">
-            <xacro:property name="tcp_z" value="0.172"/>
+        <xacro:if value="${upside_down}">
+            <!-- 0.7855 yaw similar to upside-down robot -->
+            <xacro:property name="gripper_base_rpy" value="0 0 0.7588"/>
         </xacro:if>
+        <xacro:unless value="${upside_down}">
+            <xacro:property name="gripper_base_rpy" value="0 0 0.0"/>
+        </xacro:unless>
         <xacro:unless value="${attach_to == ''}">
             <joint name="${prefix}gripper_fix" type="fixed">
                 <parent link="${attach_to}"/>
                 <child link="${prefix}xarm_gripper_base_link"/>
-                <origin xyz="${xyz}" rpy="${rpy}"/>
+                <origin xyz="0 0 0" rpy="${gripper_base_rpy}"/>
             </joint>
         </xacro:unless>
@@ -408,5 +419,5 @@
             type="fixed">
             <origin
-                xyz="0 0 ${tcp_z}"
+                xyz="0 0 ${tcp_offset_z}"
                 rpy="0 0 0"/>
             <parent

File: xarm_gripper/urdf/xarm_gripper_model.xacro (robot description, xacro)
@@ -9,10 +9,11 @@
     <xacro:include filename="$(find xarm_gripper)/urdf/xarm_gripper.gazebo.xacro"/>
     <xacro:macro name="load_gripper"
-                 params="prefix:='' attach_to:='' ns:='xarm' xyz:='0 0 0' rpy:='0 0 0' effort_control:='false'
-                 velocity_control:='false' robot_dof:=7 gripper_meshes_path:='' tcp_z:='' ">
+                 params="prefix:='' attach_to:='' ns:='xarm' effort_control:='false'
+                 velocity_control:='false' robot_dof:=7 gripper_meshes_path:='' long_finger:='false'
+                 upside_down:='false'">
         <!-- gazebo plugin -->
         <!-- <xacro:gazebo_ros_control_plugin namespace="${ns}"/> -->
-        <xacro:xarm_gripper_urdf prefix="${prefix}" attach_to="${attach_to}" xyz="${xyz}" rpy="${rpy}"
-                                 gripper_meshes_path="${gripper_meshes_path}" tcp_z="${tcp_z}" />
+        <xacro:xarm_gripper_urdf prefix="${prefix}" attach_to="${attach_to}" upside_down="${upside_down}"
+                                 long_finger="${long_finger}" gripper_meshes_path="${gripper_meshes_path}"/>
         <xacro:xarm_gripper_transmission prefix="${prefix}"
                                          hard_interface="$(eval 'EffortJointInterface' if ${effort_control} else 'VelocityJointInterface' if ${velocity_control} else 'PositionJointInterface')"/>

Commit message: fix (xarm6_gripper_moveit_config): upside_down argument push down

File: xarm_description/urdf/xarm6_with_gripper.xacro (robot description, xacro)
@@ -14,4 +14,5 @@
     <xacro:arg name="base_link_xyz" default="0 0 0"/>
     <xacro:arg name="long_finger" default="false"/>
+    <xacro:arg name="upside_down" default="false"/>
     <!---->
     <!-- load xarm6 robot -->
@@ -29,5 +30,6 @@
         <xacro:load_gripper attach_to="$(arg prefix)link_eef" effort_control="$(arg effort_control)"
                             velocity_control="$(arg velocity_control)" robot_dof="6"
-                            gripper_meshes_path="$(arg gripper_meshes_path)" long_finger="$(arg long_finger)"/>
+                            gripper_meshes_path="$(arg gripper_meshes_path)" long_finger="$(arg long_finger)"
+                            upside_down="$(arg upside_down)"/>
     </xacro:unless>
     <xacro:if value="$(arg use_gazebo_camera)">

File: xarm_gripper/urdf/xarm_gripper.urdf.xacro (robot description, xacro)
@@ -17,9 +17,9 @@
         </xacro:if>
         <xacro:if value="${upside_down}">
-            <!-- 0.7855 yaw similar to upside-down robot -->
-            <xacro:property name="gripper_base_rpy" value="0 0 0.7588"/>
+            <!-- 0.7855? yaw similar to real upside-down robot -->
+            <xacro:property name="gripper_base_rpy" value="0 0 0.7855"/>
         </xacro:if>
         <xacro:unless value="${upside_down}">
-            <xacro:property name="gripper_base_rpy" value="0 0 0.0"/>
+            <xacro:property name="gripper_base_rpy" value="0 0 0"/>
         </xacro:unless>
         <xacro:unless value="${attach_to == ''}">

Commit message: feat: tool_changer sim and real added

File: xarm_description/urdf/xarm6_with_gripper.xacro (robot description, xacro)
@@ -15,4 +15,5 @@
     <xacro:arg name="long_finger" default="false"/>
     <xacro:arg name="upside_down" default="false"/>
+    <xacro:arg name="tool_changer" default="false"/>
     <!---->
     <!-- load xarm6 robot -->
@@ -31,5 +32,5 @@
                             velocity_control="$(arg velocity_control)" robot_dof="6"
                             gripper_meshes_path="$(arg gripper_meshes_path)" long_finger="$(arg long_finger)"
-                            upside_down="$(arg upside_down)"/>
+                            upside_down="$(arg upside_down)" tool_changer="$(arg tool_changer)"/>
     </xacro:unless>
     <xacro:if value="$(arg use_gazebo_camera)">

File: xarm_gripper/urdf/xarm_gripper.urdf.xacro (robot description, xacro)
@@ -5,5 +5,6 @@
     -->
     <xacro:macro name="xarm_gripper_urdf"
-                 params="prefix:='' attach_to:='' gripper_meshes_path:='' long_finger:='false' upside_down:='false'">
+                 params="prefix:='' attach_to:='' gripper_meshes_path:='' long_finger:='false' upside_down:='false'
+                        tool_changer:='false'">
         <xacro:if value="${long_finger}">
             <xacro:property name="gripper_meshes_path" value="xarm_gripper/meshes/xarm_long_finger_assembled"/>
@@ -23,4 +24,12 @@
             <xacro:property name="gripper_base_rpy" value="0 0 0"/>
         </xacro:unless>
+        <xacro:if value="${tool_changer}">
+            <xacro:property name="drive_joint_z" value="0.077"/>
+            <xacro:property name="base_link_mesh_path" value="xarm_gripper/meshes/xarm_long_finger_tool_change_edited"/>
+        </xacro:if>
+        <xacro:unless value="${tool_changer}">
+            <xacro:property name="drive_joint_z" value="0" />
+            <xacro:property name="base_link_mesh_path" value="${gripper_meshes_path}"/>
+        </xacro:unless>
         <xacro:unless value="${attach_to == ''}">
             <joint name="${prefix}gripper_fix" type="fixed">
@@ -52,5 +61,5 @@
                 <geometry>
                     <mesh
-                        filename="package://${gripper_meshes_path}/base_link.STL"/>
+                        filename="package://${base_link_mesh_path}/base_link.STL"/>
                 </geometry>
                 <!-- <material
@@ -69,5 +78,5 @@
                 <geometry>
                     <mesh
-                        filename="package://${gripper_meshes_path}/base_link_collision.STL"/>
+                        filename="package://${base_link_mesh_path}/base_link_collision.STL"/>
                 </geometry>
             </collision>
@@ -115,5 +124,5 @@
             type="revolute">
             <origin
-                xyz="0 0.035 0.059098"
+                xyz="0 0.035 ${drive_joint_z + 0.059098}"
                 rpy="0 0 0"/>
             <parent
@@ -228,5 +237,5 @@
             type="revolute">
             <origin
-                xyz="0 0.02 0.074098"
+                xyz="0 0.02 ${drive_joint_z + 0.074098}"
                 rpy="0 0 0"/>
             <parent
@@ -285,5 +294,5 @@
             type="revolute">
             <origin
-                xyz="0 -0.035 0.059098"
+                xyz="0 -0.035 ${drive_joint_z + 0.059098}"
                 rpy="0 0 0"/>
             <parent
@@ -399,5 +408,5 @@
             type="revolute">
             <origin
-                xyz="0 -0.02 0.074098"
+                xyz="0 -0.02 ${drive_joint_z + 0.074098}"
                 rpy="0 0 0"/>
             <parent

File: xarm_gripper/urdf/xarm_gripper_model.xacro (robot description, xacro)
@@ -11,9 +11,10 @@
                  params="prefix:='' attach_to:='' ns:='xarm' effort_control:='false'
                  velocity_control:='false' robot_dof:=7 gripper_meshes_path:='' long_finger:='false'
-                 upside_down:='false'">
+                 upside_down:='false' tool_changer:='false'">
         <!-- gazebo plugin -->
         <!-- <xacro:gazebo_ros_control_plugin namespace="${ns}"/> -->
         <xacro:xarm_gripper_urdf prefix="${prefix}" attach_to="${attach_to}" upside_down="${upside_down}"
-                                 long_finger="${long_finger}" gripper_meshes_path="${gripper_meshes_path}"/>
+                                 long_finger="${long_finger}" gripper_meshes_path="${gripper_meshes_path}"
+                                 tool_changer="${tool_changer}"/>
         <xacro:xarm_gripper_transmission prefix="${prefix}"
                                          hard_interface="$(eval 'EffortJointInterface' if ${effort_control} else 'VelocityJointInterface' if ${velocity_control} else 'PositionJointInterface')"/>
