Commit message: feat: use realsense camera model
fix: fix camera's base link transformation

fix: change joint limits according to UFactory GUI

File: xarm_description/urdf/xarm6_robot_macro.xacro (robot description, xacro)
@@ -34,10 +34,10 @@
     <xacro:if value="${limited}">
       <xacro:xarm6_urdf prefix="${prefix}"
-        joint1_lower_limit="${-pi*0.99}" joint1_upper_limit="${pi*0.99}"
+        joint1_lower_limit="${-2.0*pi}" joint1_upper_limit="${2.0*pi}"
         joint2_lower_limit="${-2.059}" joint2_upper_limit="${2.0944}"
-        joint3_lower_limit="${-pi*0.99}" joint3_upper_limit="${0.19198}"
-        joint4_lower_limit="${pi*0.0}" joint4_upper_limit="${pi*2}"
+        joint3_lower_limit="${-3.927}" joint3_upper_limit="${0.19198}"
+        joint4_lower_limit="${-2.0*pi}" joint4_upper_limit="${2.0*pi}"
         joint5_lower_limit="${-1.69297}" joint5_upper_limit="${pi*0.99}"
-        joint6_lower_limit="${-2*pi*0.99}" joint6_upper_limit="${2*pi*0.99}"
+        joint6_lower_limit="${-2.0*pi}" joint6_upper_limit="${2.0*pi}"
         rs_d435i="${rs_d435i}"/>
     </xacro:if>

File: xarm_description/urdf/xarm6_with_gripper.xacro (robot description, xacro)
@@ -21,17 +21,30 @@
     <!-- Attach gripper -->
     <xacro:include filename="$(find xarm_gripper)/urdf/xarm_gripper_model.xacro"/>
-    <xacro:xarm6_robot prefix="$(arg prefix)" namespace="$(arg ros_namespace)" limited="$(arg limited)"
-                       effort_control="$(arg effort_control)" velocity_control="$(arg velocity_control)"
-                       rs_d435i="$(arg add_realsense_d435i)" rpy="$(arg base_link_rpy)" xyz="$(arg base_link_xyz)"/>
+    <xacro:xarm6_robot prefix="$(arg prefix)" namespace="$(arg ros_namespace)"
+                       limited="$(arg limited)"
+                       effort_control="$(arg effort_control)"
+                       velocity_control="$(arg velocity_control)"
+                       rs_d435i="$(arg add_realsense_d435i)" rpy="$(arg base_link_rpy)"
+                       xyz="$(arg base_link_xyz)"/>
     <xacro:if value="$(arg add_realsense_d435i)">
-        <xacro:load_gripper attach_to="$(arg prefix)link_eef" xyz="0 0 0.003" effort_control="$(arg effort_control)"
+        <xacro:load_gripper attach_to="$(arg prefix)link_eef" xyz="0 0 0.003"
+                            effort_control="$(arg effort_control)"
                             velocity_control="$(arg velocity_control)" robot_dof="6"/>
     </xacro:if>
     <xacro:unless value="$(arg add_realsense_d435i)">
-        <xacro:load_gripper attach_to="$(arg prefix)link_eef" effort_control="$(arg effort_control)"
+        <xacro:load_gripper attach_to="$(arg prefix)link_eef"
+                            effort_control="$(arg effort_control)"
                             velocity_control="$(arg velocity_control)" robot_dof="6"
-                            gripper_meshes_path="$(arg gripper_meshes_path)" long_finger="$(arg long_finger)"
+                            gripper_meshes_path="$(arg gripper_meshes_path)"
+                            long_finger="$(arg long_finger)"
                             upside_down="$(arg upside_down)" tool_changer="$(arg tool_changer)"/>
     </xacro:unless>
+    <!-- attach camera -->
+    <xacro:include filename="$(find realsense2_description)/urdf/_d435.urdf.xacro"/>
+    <xacro:sensor_d435 parent="$(arg prefix)link_eef" use_mesh="true" add_plug="false"
+                       use_nominal_extrinsics="true">
+            <origin xyz="0 -0.051 -0.0115" rpy="0 0 ${pi*(-1/2)}"/>
+<!--        <origin xyz="0 -0.051 -0.04" rpy="0 0 ${pi*(-1/2)}"/>-->
+    </xacro:sensor_d435>
     <xacro:if value="$(arg use_gazebo_camera)">
         <!-- <xacro:include filename="$(find kinect_v2)/urdf/kinect_v2.urdf.xacro" />

File: xarm_gripper/urdf/xarm_gripper.urdf.xacro (robot description, xacro)
@@ -8,5 +8,6 @@
                         tool_changer:='false'">
         <xacro:if value="${long_finger}">
-            <xacro:property name="gripper_meshes_path" value="xarm_gripper/meshes/xarm_long_finger_assembled"/>
+            <xacro:property name="gripper_meshes_path"
+                            value="xarm_gripper/meshes/xarm_long_finger_assembled"/>
             <xacro:property name="tcp_offset_z" value="0.340"/>
         </xacro:if>
@@ -26,5 +27,6 @@
         <xacro:if value="${tool_changer}">
             <xacro:property name="drive_joint_z" value="0.077"/>
-            <xacro:property name="base_link_mesh_path" value="xarm_gripper/meshes/xarm_long_finger_tool_change_edited"/>
+            <xacro:property name="base_link_mesh_path"
+                            value="xarm_gripper/meshes/xarm_long_finger_tool_change_edited"/>
             <!--            <xacro:property name="base_link_mesh_path" value="xarm_gripper/meshes/xarm_long_finger_assembled"/>-->
         </xacro:if>
@@ -41,26 +43,26 @@
         </xacro:unless>
         <link
-            name="${prefix}xarm_gripper_base_link">
-            <inertial>
-                <origin
-                    xyz="-0.00065489 -0.0018497 0.048028"
-                    rpy="0 0 0"/>
-                <mass
-                    value="0.54156"/>
-                <inertia
-                    ixx="0.00047106"
-                    ixy="3.9292E-07"
-                    ixz="2.6537E-06"
-                    iyy="0.00033072"
-                    iyz="-1.0975E-05"
-                    izz="0.00025642"/>
-            </inertial>
-            <visual>
-                <origin
-                    xyz="0 0 0"
-                    rpy="0 0 0"/>
-                <geometry>
-                    <mesh
-                        filename="package://${base_link_mesh_path}/base_link.STL"/>
+                name="${prefix}xarm_gripper_base_link">
+            <inertial>
+                <origin
+                        xyz="-0.00065489 -0.0018497 0.048028"
+                        rpy="0 0 0"/>
+                <mass
+                        value="0.54156"/>
+                <inertia
+                        ixx="0.00047106"
+                        ixy="3.9292E-07"
+                        ixz="2.6537E-06"
+                        iyy="0.00033072"
+                        iyz="-1.0975E-05"
+                        izz="0.00025642"/>
+            </inertial>
+            <visual>
+                <origin
+                        xyz="0 0 0"
+                        rpy="0 0 0"/>
+                <geometry>
+                    <mesh
+                            filename="package://${base_link_mesh_path}/base_link.STL"/>
                 </geometry>
                 <!-- <material
@@ -75,9 +77,9 @@
             <collision>
                 <origin
-                    xyz="0 0 0"
-                    rpy="0 0 0"/>
-                <geometry>
-                    <mesh
-                        filename="package://${base_link_mesh_path}/base_link_collision.STL"/>
+                        xyz="0 0 0"
+                        rpy="0 0 0"/>
+                <geometry>
+                    <mesh
+                            filename="package://${base_link_mesh_path}/base_link_collision.STL"/>
                 </geometry>
             </collision>
@@ -85,371 +87,376 @@
         <!-- add condition for camera if needed -->
         <xacro:if value="${True}">
-            <link name="camera_center">
-                <origin xyz="0 0 0" rpy="0 0 0"/>
-            </link>
-            <joint
-                name="camera_joint"
+<!--            <link name="my_camera_link">-->
+<!--                <origin xyz="0 0 0" rpy="0 0 0"/>-->
+<!--            </link>-->
+<!--            <joint-->
+<!--                    name="my_camera_joint"-->
+<!--                    type="fixed">-->
+<!--                <origin-->
+<!--                        xyz="-0.0463 -0.0467 0"-->
+<!--                        rpy="${(1.0/2)*pi} ${(2/2)*pi} ${(-1/4)*pi}"/>-->
+<!--                &lt;!&ndash; xyz="-0.0463 -0.0467 0"&ndash;&gt;-->
+<!--                &lt;!&ndash;camera image from with reversed y&ndash;&gt;-->
+<!--                &lt;!&ndash; rpy="${(1/2)*pi} ${(2/2)*pi} ${(-1/4)*pi}"/>&ndash;&gt;-->
+<!--                &lt;!&ndash; camera image for test/calibration with real-sense ros package&ndash;&gt;-->
+<!--                &lt;!&ndash; rpy="${(-0.1/2)*pi} ${(0.0/2)*pi} ${(-2.9/4)*pi}"/>&ndash;&gt;-->
+<!--                <parent-->
+<!--                        link="${prefix}xarm_gripper_base_link"/>-->
+<!--                <child-->
+<!--                        link="my_camera_link"/>-->
+<!--            </joint>-->
+        </xacro:if>
+        <link
+                name="${prefix}left_outer_knuckle">
+            <inertial>
+                <origin
+                        xyz="2.9948E-14 0.021559 0.015181"
+                        rpy="0 0 0"/>
+                <mass
+                        value="0.033618"/>
+                <inertia
+                        ixx="1.9111E-05"
+                        ixy="-1.8803E-17"
+                        ixz="-1.1002E-17"
+                        iyy="6.6256E-06"
+                        iyz="-7.3008E-06"
+                        izz="1.3185E-05"/>
+            </inertial>
+            <visual>
+                <origin
+                        xyz="0 0 0"
+                        rpy="0 0 0"/>
+                <geometry>
+                    <mesh
+                            filename="package://${gripper_meshes_path}/left_outer_knuckle.STL"/>
+                </geometry>
+                <material name="Silver">
+                    <color rgba="0.753 0.753 0.753 1.0"/>
+                </material>
+            </visual>
+            <collision>
+                <origin
+                        xyz="0 0 0"
+                        rpy="0 0 0"/>
+                <geometry>
+                    <mesh
+                            filename="package://${gripper_meshes_path}/left_outer_knuckle.STL"/>
+                </geometry>
+            </collision>
+        </link>
+        <joint
+                name="${prefix}drive_joint"
+                type="revolute">
+            <origin
+                    xyz="0 0.035 ${drive_joint_z + 0.059098}"
+                    rpy="0 0 0"/>
+            <parent
+                    link="${prefix}xarm_gripper_base_link"/>
+            <child
+                    link="${prefix}left_outer_knuckle"/>
+            <axis
+                    xyz="1 0 0"/>
+            <limit
+                    lower="0"
+                    upper="0.85"
+                    effort="50"
+                    velocity="2"/>
+        </joint>
+        <link
+                name="${prefix}left_finger">
+            <inertial>
+                <origin
+                        xyz="-2.4536E-14 -0.016413 0.029258"
+                        rpy="0 0 0"/>
+                <mass
+                        value="0.048304"/>
+                <inertia
+                        ixx="1.7493E-05"
+                        ixy="-4.2156E-19"
+                        ixz="6.9164E-18"
+                        iyy="1.7225E-05"
+                        iyz="4.6433E-06"
+                        izz="5.1466E-06"/>
+            </inertial>
+            <visual>
+                <origin
+                        xyz="0 0 0"
+                        rpy="0 0 0"/>
+                <geometry>
+                    <mesh
+                            filename="package://${gripper_meshes_path}/left_finger.STL"/>
+                </geometry>
+                <material name="Silver">
+                    <color rgba="0.753 0.753 0.753 1.0"/>
+                </material>
+            </visual>
+            <collision>
+                <origin
+                        xyz="0 0 0"
+                        rpy="0 0 0"/>
+                <geometry>
+                    <mesh
+                            filename="package://${gripper_meshes_path}/left_finger.STL"/>
+                </geometry>
+            </collision>
+        </link>
+        <joint
+                name="${prefix}left_finger_joint"
+                type="revolute">
+            <origin
+                    xyz="0 0.035465 0.042039"
+                    rpy="0 0 0"/>
+            <parent
+                    link="${prefix}left_outer_knuckle"/>
+            <child
+                    link="${prefix}left_finger"/>
+            <axis
+                    xyz="-1 0 0"/>
+            <limit
+                    lower="0"
+                    upper="0.85"
+                    effort="50"
+                    velocity="2"/>
+            <mimic joint="${prefix}drive_joint" multiplier="1" offset="0"/>
+        </joint>
+        <link
+                name="${prefix}left_inner_knuckle">
+            <inertial>
+                <origin
+                        xyz="1.86600784687907E-06 0.0220467847633621 0.0261334672830885"
+                        rpy="0 0 0"/>
+                <mass
+                        value="0.0230125781256706"/>
+                <inertia
+                        ixx="6.09490024271906E-06"
+                        ixy="6.06651326160071E-11"
+                        ixz="7.19102670500635E-11"
+                        iyy="6.01955084375188E-06"
+                        iyz="-2.75316812991721E-06"
+                        izz="5.07862004479903E-06"/>
+            </inertial>
+            <visual>
+                <origin
+                        xyz="0 0 0"
+                        rpy="0 0 0"/>
+                <geometry>
+                    <mesh
+                            filename="package://${gripper_meshes_path}/left_inner_knuckle.STL"/>
+                </geometry>
+                <material name="Silver">
+                    <color rgba="0.753 0.753 0.753 1.0"/>
+                </material>
+            </visual>
+            <collision>
+                <origin
+                        xyz="0 0 0"
+                        rpy="0 0 0"/>
+                <geometry>
+                    <mesh
+                            filename="package://${gripper_meshes_path}/left_inner_knuckle.STL"/>
+                </geometry>
+            </collision>
+        </link>
+        <joint
+                name="${prefix}left_inner_knuckle_joint"
+                type="revolute">
+            <origin
+                    xyz="0 0.02 ${drive_joint_z + 0.074098}"
+                    rpy="0 0 0"/>
+            <parent
+                    link="${prefix}xarm_gripper_base_link"/>
+            <child
+                    link="${prefix}left_inner_knuckle"/>
+            <axis
+                    xyz="1 0 0"/>
+            <limit
+                    lower="0"
+                    upper="0.85"
+                    effort="50"
+                    velocity="2"/>
+            <mimic joint="${prefix}drive_joint" multiplier="1" offset="0"/>
+        </joint>
+        <link
+                name="${prefix}right_outer_knuckle">
+            <inertial>
+                <origin
+                        xyz="-3.1669E-14 -0.021559 0.015181"
+                        rpy="0 0 0"/>
+                <mass
+                        value="0.033618"/>
+                <inertia
+                        ixx="1.9111E-05"
+                        ixy="-1.8789E-17"
+                        ixz="1.0986E-17"
+                        iyy="6.6256E-06"
+                        iyz="7.3008E-06"
+                        izz="1.3185E-05"/>
+            </inertial>
+            <visual>
+                <origin
+                        xyz="0 0 0"
+                        rpy="0 0 0"/>
+                <geometry>
+                    <mesh
+                            filename="package://${gripper_meshes_path}/right_outer_knuckle.STL"/>
+                </geometry>
+                <material name="Silver">
+                    <color rgba="0.753 0.753 0.753 1.0"/>
+                </material>
+            </visual>
+            <collision>
+                <origin
+                        xyz="0 0 0"
+                        rpy="0 0 0"/>
+                <geometry>
+                    <mesh
+                            filename="package://${gripper_meshes_path}/right_outer_knuckle.STL"/>
+                </geometry>
+            </collision>
+        </link>
+        <joint
+                name="${prefix}right_outer_knuckle_joint"
+                type="revolute">
+            <origin
+                    xyz="0 -0.035 ${drive_joint_z + 0.059098}"
+                    rpy="0 0 0"/>
+            <parent
+                    link="${prefix}xarm_gripper_base_link"/>
+            <child
+                    link="${prefix}right_outer_knuckle"/>
+            <axis
+                    xyz="-1 0 0"/>
+            <limit
+                    lower="0"
+                    upper="0.85"
+                    effort="50"
+                    velocity="2"/>
+            <mimic joint="${prefix}drive_joint" multiplier="1" offset="0"/>
+        </joint>
+        <link
+                name="${prefix}right_finger">
+            <inertial>
+                <origin
+                        xyz="2.5618E-14 0.016413 0.029258"
+                        rpy="0 0 0"/>
+                <mass
+                        value="0.048304"/>
+                <inertia
+                        ixx="1.7493E-05"
+                        ixy="-5.0014E-19"
+                        ixz="-7.5079E-18"
+                        iyy="1.7225E-05"
+                        iyz="-4.6435E-06"
+                        izz="5.1466E-06"/>
+            </inertial>
+            <visual>
+                <origin
+                        xyz="0 0 0"
+                        rpy="0 0 0"/>
+                <geometry>
+                    <mesh
+                            filename="package://${gripper_meshes_path}/right_finger.STL"/>
+                </geometry>
+                <material name="Silver">
+                    <color rgba="0.753 0.753 0.753 1.0"/>
+                </material>
+            </visual>
+            <collision>
+                <origin
+                        xyz="0 0 0"
+                        rpy="0 0 0"/>
+                <geometry>
+                    <mesh
+                            filename="package://${gripper_meshes_path}/right_finger.STL"/>
+                </geometry>
+            </collision>
+        </link>
+        <joint
+                name="${prefix}right_finger_joint"
+                type="revolute">
+            <origin
+                    xyz="0 -0.035465 0.042039"
+                    rpy="0 0 0"/>
+            <parent
+                    link="${prefix}right_outer_knuckle"/>
+            <child
+                    link="${prefix}right_finger"/>
+            <axis
+                    xyz="1 0 0"/>
+            <limit
+                    lower="0"
+                    upper="0.85"
+                    effort="50"
+                    velocity="2"/>
+            <mimic joint="${prefix}drive_joint" multiplier="1" offset="0"/>
+        </joint>
+        <link
+                name="${prefix}right_inner_knuckle">
+            <inertial>
+                <origin
+                        xyz="1.866E-06 -0.022047 0.026133"
+                        rpy="0 0 0"/>
+                <mass
+                        value="0.023013"/>
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