Commit message: feat(vacuum_gripper): attach camera

File: xarm_description/urdf/xarm6_with_vacuum_gripper.xacro (robot description, xacro)
@@ -1,22 +1,35 @@
 <?xml version='1.0' encoding='utf-8'?>
 <robot xmlns:xacro="http://ros.org/wiki/xacro" name="xarm6">
-  <xacro:arg name="prefix" default=""/>
-  <xacro:arg name="ros_namespace" default="xarm"/>
-  <xacro:arg name="limited" default="false"/>
-  <xacro:arg name="effort_control" default="false"/>
-  <xacro:arg name="velocity_control" default="false"/>
-  <!-- To add realsense d435i and vacuum gripper, set 'add_realsense_d435i' = true -->
-  <xacro:arg name="add_realsense_d435i" default="false"/>
-  <!-- load xarm6 robot -->
-  <xacro:include filename="$(find xarm_description)/urdf/xarm6_robot_macro.xacro" />
-  <!-- Attach gripper -->
-  <xacro:include filename="$(find xarm_description)/urdf/xarm_vacuum_gripper.urdf.xacro" />
-  <!-- <xacro:load_gripper attach_to="$(arg prefix)link6" /> -->
-  <xacro:xarm6_robot prefix="$(arg prefix)" namespace="$(arg ros_namespace)" limited="$(arg limited)" effort_control="$(arg effort_control)" velocity_control="$(arg velocity_control)" rs_d435i="$(arg add_realsense_d435i)" />
-  <xacro:if value="$(arg add_realsense_d435i)">
-    <xacro:xarm_vacuum_gripper_urdf attach_to="$(arg prefix)link_eef" xyz="0 0 0.003" effort_control="$(arg effort_control)" velocity_control="$(arg velocity_control)" />
-  </xacro:if>
-  <xacro:unless value="$(arg add_realsense_d435i)">
-    <xacro:xarm_vacuum_gripper_urdf attach_to="$(arg prefix)link_eef" effort_control="$(arg effort_control)" velocity_control="$(arg velocity_control)" />
-  </xacro:unless>
+    <xacro:arg name="prefix" default=""/>
+    <xacro:arg name="ros_namespace" default="xarm"/>
+    <xacro:arg name="limited" default="false"/>
+    <xacro:arg name="effort_control" default="false"/>
+    <xacro:arg name="velocity_control" default="false"/>
+    <!-- To add realsense d435i and vacuum gripper, set 'add_realsense_d435i' = true -->
+    <xacro:arg name="add_realsense_d435i" default="false"/>
+    <!-- load xarm6 robot -->
+    <xacro:include filename="$(find xarm_description)/urdf/xarm6_robot_macro.xacro"/>
+    <!-- Attach gripper -->
+    <xacro:include filename="$(find xarm_description)/urdf/xarm_vacuum_gripper.urdf.xacro"/>
+    <!-- <xacro:load_gripper attach_to="$(arg prefix)link6" /> -->
+    <!-- attach camera -->
+    <xacro:include filename="$(find realsense2_description)/urdf/_d435.urdf.xacro"/>
+    <xacro:sensor_d435 parent="$(arg prefix)link_eef" use_mesh="true" add_plug="false"
+                       use_nominal_extrinsics="true">
+        <origin xyz="-0.0365 -0.0365 -0.0115" rpy="0 0 ${pi*(-3/4)}"/>
+    </xacro:sensor_d435>
+    <xacro:xarm6_robot prefix="$(arg prefix)" namespace="$(arg ros_namespace)"
+                       limited="$(arg limited)" effort_control="$(arg effort_control)"
+                       velocity_control="$(arg velocity_control)"
+                       rs_d435i="$(arg add_realsense_d435i)"/>
+    <xacro:if value="$(arg add_realsense_d435i)">
+        <xacro:xarm_vacuum_gripper_urdf attach_to="$(arg prefix)link_eef" xyz="0 0 0.003"
+                                        effort_control="$(arg effort_control)"
+                                        velocity_control="$(arg velocity_control)"/>
+    </xacro:if>
+    <xacro:unless value="$(arg add_realsense_d435i)">
+        <xacro:xarm_vacuum_gripper_urdf attach_to="$(arg prefix)link_eef"
+                                        effort_control="$(arg effort_control)"
+                                        velocity_control="$(arg velocity_control)"/>
+    </xacro:unless>
 </robot>
