Commit message: fix: rpy for joint eef instead of gripper urdf

File: xarm_description/urdf/xarm6.urdf.xacro (robot description, xacro)
@@ -322,5 +322,5 @@
     <origin
       xyz="0 0 0"
-      rpy="0 0 0" />
+      rpy="0 0 0.7855" />
     <parent
       link="${prefix}link6" />

File: xarm_description/urdf/xarm6_with_gripper.xacro (robot description, xacro)
@@ -44,5 +44,6 @@
     <xacro:sensor_d435 parent="$(arg prefix)link_eef" use_mesh="true" add_plug="false"
                        use_nominal_extrinsics="true">
-            <origin xyz="0 -0.051 -0.0115" rpy="0 0 ${pi*(-1/2)}"/>
+        <origin xyz="-0.0365 -0.0365 -0.0115" rpy="0 0 ${pi*(-3/4)}"/>
+<!--            <origin xyz="0 -0.051 -0.0115" rpy="0 0 ${pi*(-1/2)}"/>-->
 <!--        <origin xyz="0 -0.051 -0.04" rpy="0 0 ${pi*(-1/2)}"/>-->
     </xacro:sensor_d435>

File: xarm_gripper/urdf/xarm_gripper.urdf.xacro (robot description, xacro)
@@ -18,11 +18,11 @@
             <xacro:property name="gripper_meshes_path" value="xarm_gripper/meshes"/>
         </xacro:if>
-        <xacro:if value="${upside_down}">
-            <!-- 0.7855? yaw similar to real upside-down robot -->
-            <xacro:property name="gripper_base_rpy" value="0 0 0.7855"/>
-        </xacro:if>
-        <xacro:unless value="${upside_down}">
-            <xacro:property name="gripper_base_rpy" value="0 0 0.7855"/>
-        </xacro:unless>
+<!--        <xacro:if value="${upside_down}">-->
+<!--            &lt;!&ndash; 0.7855? yaw similar to real upside-down robot &ndash;&gt;-->
+<!--            <xacro:property name="gripper_base_rpy" value="0 0 0.7855"/>-->
+<!--        </xacro:if>-->
+<!--        <xacro:unless value="${upside_down}">-->
+<!--            <xacro:property name="gripper_base_rpy" value="0 0 0.7855"/>-->
+<!--        </xacro:unless>-->
         <xacro:if value="${tool_changer}">
             <xacro:property name="drive_joint_z" value="0.077"/>
@@ -39,5 +39,5 @@
                 <parent link="${attach_to}"/>
                 <child link="${prefix}xarm_gripper_base_link"/>
-                <origin xyz="0 0 0" rpy="${gripper_base_rpy}"/>
+                <origin xyz="0 0 0" rpy="0 0 0"/>
             </joint>
         </xacro:unless>
