Commit message: fix (xarm_gazebo): upside_down argument pass down
refactor (xarm_gazebo): redundant stl files removed

fix (xarm_gazebo): added simplified version of base_link_collision.stl

fix (xarm_gazebo): tcp offset fixed for tool_changer

File: xarm_gripper/urdf/xarm_gripper.urdf.xacro (robot description, xacro)
@@ -27,4 +27,5 @@
             <xacro:property name="drive_joint_z" value="0.077"/>
             <xacro:property name="base_link_mesh_path" value="xarm_gripper/meshes/xarm_long_finger_tool_change_edited"/>
+<!--            <xacro:property name="base_link_mesh_path" value="xarm_gripper/meshes/xarm_long_finger_assembled"/>-->
         </xacro:if>
         <xacro:unless value="${tool_changer}">
@@ -428,5 +429,5 @@
             type="fixed">
             <origin
-                xyz="0 0 ${tcp_offset_z}"
+                xyz="0 0 ${tcp_offset_z + drive_joint_z}"
                 rpy="0 0 0"/>
             <parent

Commit message: config: eef base_link yaw edited according to new setup

File: xarm_gripper/urdf/xarm_gripper.urdf.xacro (robot description, xacro)
@@ -19,5 +19,5 @@
         <xacro:if value="${upside_down}">
             <!-- 0.7855? yaw similar to real upside-down robot -->
-            <xacro:property name="gripper_base_rpy" value="0 0 0.7855"/>
+            <xacro:property name="gripper_base_rpy" value="0 0 0.0"/>
         </xacro:if>
         <xacro:unless value="${upside_down}">

Commit message: feat (robot_model): camera TF added

File: xarm_gripper/urdf/xarm_gripper.urdf.xacro (robot description, xacro)
@@ -27,8 +27,8 @@
             <xacro:property name="drive_joint_z" value="0.077"/>
             <xacro:property name="base_link_mesh_path" value="xarm_gripper/meshes/xarm_long_finger_tool_change_edited"/>
-<!--            <xacro:property name="base_link_mesh_path" value="xarm_gripper/meshes/xarm_long_finger_assembled"/>-->
+            <!--            <xacro:property name="base_link_mesh_path" value="xarm_gripper/meshes/xarm_long_finger_assembled"/>-->
         </xacro:if>
         <xacro:unless value="${tool_changer}">
-            <xacro:property name="drive_joint_z" value="0" />
+            <xacro:property name="drive_joint_z" value="0"/>
             <xacro:property name="base_link_mesh_path" value="${gripper_meshes_path}"/>
         </xacro:unless>
@@ -83,4 +83,20 @@
             </collision>
         </link>
+        <xacro:if value="${tool_changer}">
+            <link name="camera_center">
+                <origin xyz="0 0 0" rpy="0 0 0"/>
+            </link>
+            <joint
+                name="camera_joint"
+                type="fixed">
+                <origin
+                    xyz="-0.0463 -0.0467 0"
+                    rpy="0 0 ${(3/4)*pi}"/>
+                <parent
+                    link="${prefix}xarm_gripper_base_link"/>
+                <child
+                    link="camera_center"/>
+            </joint>
+        </xacro:if>
         <link
             name="${prefix}left_outer_knuckle">

Commit message: config (urdf): gripper yaw changed by 90 degree according to the new setup of real robot

File: xarm_gripper/urdf/xarm_gripper.urdf.xacro (robot description, xacro)
@@ -19,8 +19,8 @@
         <xacro:if value="${upside_down}">
             <!-- 0.7855? yaw similar to real upside-down robot -->
-            <xacro:property name="gripper_base_rpy" value="0 0 0.0"/>
+            <xacro:property name="gripper_base_rpy" value="0 0 0.7855"/>
         </xacro:if>
         <xacro:unless value="${upside_down}">
-            <xacro:property name="gripper_base_rpy" value="0 0 0"/>
+            <xacro:property name="gripper_base_rpy" value="0 0 0.7855"/>
         </xacro:unless>
         <xacro:if value="${tool_changer}">
